Commit message: fix:ros2 control车轮的速度控制接口换成了effort接口

File: src/balance_car_description/urdf/two_wheel_balance_65mm.urdf.xacro (robot description, xacro)
@@ -16,7 +16,7 @@
   <xacro:property name="body_length" value="0.085"/>
   <xacro:property name="body_width" value="0.054"/>
-  <xacro:property name="body_height" value="0.130"/>
+  <xacro:property name="body_height" value="0.090"/>
   <xacro:property name="body_mass" value="0.420"/>
-  <xacro:property name="body_com_z" value="0.075"/>
+  <xacro:property name="body_com_z" value="0.045"/>
   <!-- Internal components represented as separate fixed masses. -->
   <xacro:property name="motor_radius" value="0.012"/>
@@ -25,5 +25,5 @@
   <xacro:property name="motor_y" value="${wheel_separation / 2.0 - wheel_width / 2.0 - motor_length / 2.0}"/>
   <xacro:property name="battery_x" value="-0.010"/>
-  <xacro:property name="battery_z" value="0.035"/>
+  <xacro:property name="battery_z" value="0.025"/>
   <xacro:property name="battery_length" value="0.052"/>
   <xacro:property name="battery_width" value="0.034"/>
@@ -31,5 +31,5 @@
   <xacro:property name="battery_mass" value="0.085"/>
   <xacro:property name="board_x" value="0.008"/>
-  <xacro:property name="board_z" value="0.110"/>
+  <xacro:property name="board_z" value="0.070"/>
   <xacro:property name="board_length" value="0.055"/>
   <xacro:property name="board_width" value="0.038"/>
@@ -37,5 +37,5 @@
   <xacro:property name="board_mass" value="0.025"/>
   <xacro:property name="imu_x" value="0.010"/>
-  <xacro:property name="imu_z" value="0.138"/>
+  <xacro:property name="imu_z" value="0.090"/>
   <xacro:property name="imu_length" value="0.018"/>
   <xacro:property name="imu_width" value="0.018"/>
@@ -280,6 +280,6 @@
   <gazebo reference="left_wheel_link">
     <material>Gazebo/Black</material>
-    <mu1>1.45</mu1>
-    <mu2>0.85</mu2>
+    <mu1>1.0</mu1>
+    <mu2>0.6</mu2>
     <kp>1000000.0</kp>
     <kd>4.0</kd>
@@ -289,6 +289,6 @@
   <gazebo reference="right_wheel_link">
     <material>Gazebo/Black</material>
-    <mu1>1.45</mu1>
-    <mu2>0.85</mu2>
+    <mu1>1.0</mu1>
+    <mu2>0.6</mu2>
     <kp>1000000.0</kp>
     <kd>4.0</kd>
@@ -387,6 +387,11 @@
         <param name="max">${wheel_velocity_limit}</param>
       </command_interface>
+      <command_interface name="effort">
+        <param name="min">${-wheel_effort_limit}</param>
+        <param name="max">${wheel_effort_limit}</param>
+      </command_interface>
       <state_interface name="position"/>
       <state_interface name="velocity"/>
+      <state_interface name="effort"/>
       <param name="mechanical_reduction">${motor_gear_ratio}</param>
     </joint>
@@ -396,6 +401,11 @@
         <param name="max">${wheel_velocity_limit}</param>
       </command_interface>
+      <command_interface name="effort">
+        <param name="min">${-wheel_effort_limit}</param>
+        <param name="max">${wheel_effort_limit}</param>
+      </command_interface>
       <state_interface name="position"/>
       <state_interface name="velocity"/>
+      <state_interface name="effort"/>
       <param name="mechanical_reduction">${motor_gear_ratio}</param>
     </joint>

Commit message: 直立环参数：修正直立时的角度;不加入速度环，不可能站立不动保持平衡。

File: src/balance_car_description/urdf/two_wheel_balance_65mm.urdf.xacro (robot description, xacro)
@@ -24,5 +24,5 @@
   <xacro:property name="motor_mass" value="0.055"/>
   <xacro:property name="motor_y" value="${wheel_separation / 2.0 - wheel_width / 2.0 - motor_length / 2.0}"/>
-  <xacro:property name="battery_x" value="-0.010"/>
+  <xacro:property name="battery_x" value="0.0"/>
   <xacro:property name="battery_z" value="0.025"/>
   <xacro:property name="battery_length" value="0.052"/>
@@ -315,5 +315,5 @@
            降到 200 Hz 后 Python rclpy 单线程 executor 压力小很多，
            且仍是控制率 200 Hz 的 1x，足够 PD 计算。-->
-      <update_rate>200</update_rate>
+      <update_rate>400</update_rate>
       <visualize>false</visualize>
       <imu>
